File: SMD/Session_02_02/Blinky/Blinky.kicad_pcb (KiCad board)
At the start: 2 copper layers, 12 parts, among them U1 TLC551CD‎

Commit message: Corrections to the switch footprint
Changed lines of the file:
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@@
     (fp_rect (start -2 -5.499999) (end -0.5 -4) (layer "F.SilkS") (width 0.1524) (fill none))
     (fp_rect (start -3.5 -5.5) (end 3.5 1) (layer "F.CrtYd") (width 0.01) (fill none))
-    (pad "" np_thru_hole circle (at -1.25 -2.75) (size 0.8 0.8) (drill 0.8) (layers F&B.Cu *.Mask))
-    (pad "" np_thru_hole circle (at 1.25 -2.75) (size 0.8 0.8) (drill 0.8) (layers F&B.Cu *.Mask))
+    (pad "" np_thru_hole circle (at -1.5 -2.75) (size 0.8 0.8) (drill 0.8) (layers F&B.Cu *.Mask))
+    (pad "" np_thru_hole circle (at 1.5 -2.75) (size 0.8 0.8) (drill 0.8) (layers F&B.Cu *.Mask))
     (pad "1" smd roundrect (at -2.5 0) (size 1 2) (layers "F.Cu" "F.Paste" "F.Mask") (roundrect_rratio 0.25)
       (net 4 "Net-(C2-Pad1)") (pinfunction "A") (pintype "passive"))
